Commit message: Update 2R_planar_robot.urdf

File: Part3/Subpart2/2R_planar_robot.urdf (robot description, URDF)
Before this commit: robot 2R_robot, 3 links, 2 joints
Links:
- added link link3; visual sphere radius=0.05
Joints:
- added joint joint3: type fixed, parent link2, child link3, origin xyz=0 0 1.05, axis 0 0 0
